File: LIN-Controller1.1.sch (KiCad schematic (older format))
At the start: 42 parts, among them CON1 BARREL_JACK, J1 SWD_HEADER, J2 1881451_LIN, SW1 TL9210, SW2 TL9210, SW3 TL9210, SW4 TL9210, SW5 TSWA3NCD23LFS_, U1 SAMC21E-A, U2 2SC5662, U3 LM2675, U4 2SC5662, U5 2SC5662, U6 2SC5662, U7 ATA663211

Commit message: Added files via upload
Parts:
- C1: symbol C -> C-RESCUE-LIN-Controller1.1; MFG P/N (none) -> F380J476MMAAXEH3
- C2, C4, C5: symbol C -> C-RESCUE-LIN-Controller1.1; MFG P/N (none) -> LLL185R71A104MA01L
- C3: symbol C -> C-RESCUE-LIN-Controller1.1; MFG P/N (none) -> 6TPH100MAEA
- C7, C8, C9: symbol C -> C-RESCUE-LIN-Controller1.1
- D1, D3, D4, D5: MFG P/N (none) -> HDSM-283L
- D2: MFG P/N (none) -> 1N5819HW-7-F
- J1: MFG P/N (none) -> M50-3500542
- L1: MFG P/N (none) -> SRR0805-330Y
- R1, R6, R7: symbol R -> R-RESCUE-LIN-Controller1.1; MFG P/N (none) -> CRCW120610K0FKEA
- R15, R16, R19, R20, R21: symbol R -> R-RESCUE-LIN-Controller1.1
- R2, R3, R4, R5: symbol R -> R-RESCUE-LIN-Controller1.1; MFG P/N (none) -> ERJ-1GEJ331C
- SW5: MFG P/N (none) -> TSWA3NCD23LFS
- U2, U4, U5, U6: MFG P/N (none) -> 2SC5662T2LP
- U3: MFG P/N (none) -> LM2675MX-ADJ/NOPB
Connections:
- net 3V3: now also C3.1, R6.1
Other:
- note removed: "LIN Bus Interface"
- note removed: "LIN Interfacing\nSERCOMOP0 Pin 5 EN\nSERCOMOP1 Pin6 TXD\nSERCOMOP2 Pin7 RXD\n\nDISPLAYS\nPA16 Pin17 Element 'g'\nPA17 Pin18 Element 'f'\nPA18 Pin19 Element 'e'\nPA19 Pin20 Element 'd'\nPA20 Pin21 Element 'c'\nPA21 Pin22 Element 'b'\nPA22 Pin23 Element 'a'\nPA23 Pin24 Decimal Point\nPA14 Pin15 1000's display select\nPA15 Pin16 100's display select\nPA27 Pin26 10's display select\nPA28 Pin27 1's di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"
- note removed: "Power Supply"
- note removed: "Programmimng Connector"
- note removed: "SAMC21 I/O Port Allocations"
- moved on the sheet: C3
